File: pathFinder.kicad_pcb (KiCad board)
At the start: 2 copper layers, 8 parts, among them SW1 SW_Push, SW2 SW_Push, U1 XIAO-RP2040-DIP

Commit message: pushed
Other:
- board outline added: 79 x 48 mm
Changed lines of the file:
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@@
 			(outputformat 1)
 			(mirror no)
-			(drillshape 1)
+			(drillshape 0)
 			(scaleselection 1)
-			(outputdirectory "")
+			(outputdirectory "../newgrb/")
 		)
 	)
@@
 		)
 	)
+	(gr_line
+		(start 121.5 104.029411)
+		(end 121.5 105)
+		(stroke
+			(width 0.05)
+			(type default)
+		)
+		(layer "Edge.Cuts")
+	)
+	(gr_arc
+		(start 119.029325 60.021993)
+		(mid 120.488231 61.759659)
+		(end 121.028979 63.963174)
+		(stroke
+			(width 0.05)
+			(type default)
+		)
+		(layer "Edge.Cuts")
+	)
+	(gr_line
+		(start 185.5 88.5)
+		(end 189 88.5)
+		(stroke
+			(width 0.05)
+			(type default)
+		)
+		(layer "Edge.Cuts")
+	)
+	(gr_line
+		(start 121.5 105)
+		(end 180.5 105)
+		(stroke
+			(width 0.05)
+			(type default)
+		)
+		(layer "Edge.Cuts")
+	)
+	(gr_line
+		(start 189.031645 57.468555)
+		(end 115 57)
+		(stroke
+			(width 0.05)
+			(type default)
+		)
+		(layer "Edge.Cuts")
+	)
+	(gr_arc
+		(start 189.031645 57.468555)
+		(mid 192.546721 58.944124)
+		(end 194 62.468455)
+		(stroke
+			(width 0.05)
+			(type default)
+		)
+		(layer "Edge.Cuts")
+	)
+	(gr_line
+		(start 194 83.5)
+		(end 194 62.468455)
+		(stroke
+			(width 0.05)
+			(type default)
+		)
+		(layer "Edge.Cuts")
+	)
+	(gr_line
+		(start 121.028979 63.963174)
+		(end 121.499654 103.970592)
+		(stroke
+			(width 0.05)
+			(type default)
+		)
+		(layer "Edge.Cuts")
+	)
+	(gr_arc
+		(start 185.5 100)
+		(mid 184.035534 103.535534)
+		(end 180.5 105)
+		(stroke
+			(width 0.05)
+			(type default)
+		)
+		(layer "Edge.Cuts")
+	)
+	(gr_arc
+		(start 194 83.5)
+		(mid 192.535534 87.035534)
+		(end 189 88.5)
+		(stroke
+			(width 0.05)
+			(type default)
+		)
+		(layer "Edge.Cuts")
+	)
+	(gr_line
+		(start 115 57)
+		(end 119.029325 60.021993)
+		(stroke
+			(width 0.05)
+			(type default)
+		)
+		(layer "Edge.Cuts")
+	)
+	(gr_line
+		(start 185.5 100)
+		(end 185.5 88.5)
+		(stroke
+			(width 0.05)
+			(type default)
+		)
+		(layer "Edge.Cuts")
+	)
+	(gr_arc
+		(start 121.499654 103.970592)
+		(mid 121.499914 104.000001)
+		(end 121.5 104.029411)
+		(stroke
+			(width 0.05)
+			(type default)
+		)
+		(layer "Edge.Cuts")
+	)
 	(segment
